File: circuits/pcb/HAT/HAT_1/HAT_1.kicad_sch (KiCad schematic)
At the start: 11 parts, among them J1 Raspberry pi 5 GPIOs, J12 power input, J2 motor1, J3 motor1, J4 Conn_01x16_Pin, J5 motor2, J7 motor2, U1 ESP32-DEVKITC-32D, U2 L293D, U3 L293D

Commit message: ..
Parts:
- removed D1: LED, LED_THT:LED_D5.0mm, symbol Device:LED
- removed J4: Conn_01x16_Pin, Connector_PinHeader_2.54mm:PinHeader_1x16_P2.54mm_Vertical, symbol Connector:Conn_01x16_Pin
- added J4: Conn_01x01_Pin, Connector_PinHeader_2.54mm:PinHeader_1x01_P2.54mm_Vertical, symbol Connector:Conn_01x01_Pin
- added J6: Conn_01x17_Pin, Connector_PinHeader_2.54mm:PinHeader_1x17_P2.54mm_Vertical, symbol Connector:Conn_01x17_Pin
Connections:
- net +5V: now also J6.1 (Pin_1)
- net ECHO 1: now also J6.17 (Pin_17)
- net ECHO 2: now also J6.16 (Pin_16)
- net ECHO 3: now also J6.15 (Pin_15)
- net ECHO 4: now also J6.14 (Pin_14)
- net ECHO 5: now also J6.13 (Pin_13)
- net GND: now also J6.2 (Pin_2)
- net GPS TX: now also J6.5 (Pin_5)
- net MQ135 A0: now also J6.6 (Pin_6)
- net MQ9 A0: now also J6.7 (Pin_7)
- net TRIG 1: now also J6.12 (Pin_12)
- net TRIG 2: now also J6.11 (Pin_11)
- net TRIG 3: now also J6.10 (Pin_10)
- net TRIG 4: now also J6.9 (Pin_9)
- net TRIG 5: now also J6.8 (Pin_8)
- net TH_CAM SCL: now reaches U1.J3-16 (IO15)
- net TH_CAM SCL: now also J6.3 (Pin_3)
- net at U1.J2-1 (3V3): now also J4.1 (Pin_1)
- net GPS RX renamed TH_CAM SDA
- net TH_CAM SDA: now also J6.4 (Pin_4)
- no-connect marks 94 -> 93
Other:
- title: (none) -> Industrial Inspection Bot
