File: circuits/pcb/HAT/HAT_2/HAT_2.kicad_pcb (KiCad board)
At the start: 2 copper layers, 64.4 x 54.4 mm, 26 parts, among them J1 Conn_01x16_Pin, J10 MQ-135, J13 USB, J14 MQ-9, J4 US 3, J5 US 2, J6 US 1, J7 GPS, J8 US 5, J9 US 4

Commit message: ..
Parts:
- removed 1K7, 2K8: R, Resistor_THT:R_Axial_DIN0207_L6.3mm_D2.5mm_P7.62mm_Horizontal
- removed J7: GPS, Connector_PinHeader_2.54mm:PinHeader_1x04_P2.54mm_Vertical
- added J11: GPS, Connector_PinHeader_2.54mm:PinHeader_1x03_P2.54mm_Vertical, F.Cu at (145.4, 63.5)
- added J2: Conn_01x17_Pin, Connector_PinHeader_2.54mm:PinHeader_1x17_P2.54mm_Vertical, F.Cu at (127.0, 68.3)
- added J3: Thermal Cam, Connector_PinHeader_2.54mm:PinHeader_1x04_P2.54mm_Vertical, F.Cu at (136.2, 51.3)
- J1: value Conn_01x16_Pin -> 3.3V; footprint Connector_PinSocket_2.54mm:PinSocket_1x16_P2.54mm_Vertical -> Connector_PinHeader_2.54mm:PinHeader_1x01_P2.54mm_Vertical
- moved J4 85.0 mm to (140.8, 51.3), turned to 0 degrees
- moved J5 76.6 mm to (145.4, 51.3), turned to 0 degrees
- moved 1K1 75.1 mm to (82.4, 64.5)
- moved 1K8 74.9 mm to (82.7, 99.0)
- moved 1K2 74.6 mm to (82.7, 70.2)
- moved 1K3 74.3 mm to (82.7, 75.8)
- moved 1K4 74.0 mm to (82.7, 81.5)
- moved 1K5 73.7 mm to (82.7, 87.2)
- moved 2K1 73.7 mm to (95.9, 64.5)
- moved 1K6 73.5 mm to (82.7, 92.8)
- moved 2K2 73.1 mm to (96.2, 70.2)
- moved 2K3 72.7 mm to (96.2, 76.0)
- moved 2K4 72.4 mm to (96.2, 81.8)
- moved 2K5 72.1 mm to (96.2, 87.5)
- moved 2K6 71.8 mm to (96.2, 93.2)
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Connections:
- J1 pad 1: +5V -> Net-(J1-Pin_1)
Other:
- board size 64.4 x 54.4 mm -> 65 x 57 mm
