File: circuits/pcb/HAT/HAT_2/HAT_2.kicad_sch (KiCad schematic)
At the start: 26 parts, among them J1 Conn_01x16_Pin, J10 MQ-135, J13 USB, J14 MQ-9, J4 US 3, J5 US 2, J6 US 1, J7 GPS, J8 US 5, J9 US 4

Commit message: ..
Parts:
- removed 1K7, 2K8: R, Resistor_THT:R_Axial_DIN0207_L6.3mm_D2.5mm_P7.62mm_Horizontal, symbol Device:R
- removed J1: Conn_01x16_Pin, Connector_PinSocket_2.54mm:PinSocket_1x16_P2.54mm_Vertical, symbol Connector:Conn_01x16_Pin
- removed J7: GPS, Connector_PinHeader_2.54mm:PinHeader_1x04_P2.54mm_Vertical, symbol Connector:Conn_01x04_Pin
- added J1: 3.3V, Connector_PinHeader_2.54mm:PinHeader_1x01_P2.54mm_Vertical, symbol Connector:Conn_01x01_Pin
- added J11: GPS, Connector_PinHeader_2.54mm:PinHeader_1x03_P2.54mm_Vertical, symbol Connector:Conn_01x03_Pin
- added J2: Conn_01x17_Pin, Connector_PinHeader_2.54mm:PinHeader_1x17_P2.54mm_Vertical, symbol Connector:Conn_01x17_Pin
- added J3: Thermal Cam, Connector_PinHeader_2.54mm:PinHeader_1x04_P2.54mm_Vertical, symbol Connector:Conn_01x04_Pin
Connections:
- net +5V: now also J2.1 (Pin_1), J3.1 (Pin_1)
- net ECHO 1: now also J2.17 (Pin_17)
- net ECHO 2: now also J2.16 (Pin_16)
- net ECHO 3: now also J2.15 (Pin_15)
- net ECHO 4: now also J2.14 (Pin_14)
- net ECHO 5: now also J2.13 (Pin_13)
- net GND: now also J11.2 (Pin_2), J2.2 (Pin_2), J3.2 (Pin_2)
- net GPS TX: now also J11.3 (Pin_3), J2.5 (Pin_5)
- net MQ135 A0: now also J2.6 (Pin_6)
- net MQ9 A0: now also J2.7 (Pin_7)
- net TRIG 1: now also J2.12 (Pin_12)
- net TRIG 2: now also J2.11 (Pin_11)
- net TRIG 3: now also J2.10 (Pin_10)
- net TRIG 4: now also J2.9 (Pin_9)
- net TRIG 5: now also J2.8 (Pin_8)
- new net: J1.1 (Pin_1), J11.1 (Pin_1)
- new net TH_CAM SCL: J2.3 (Pin_3), J3.4 (Pin_4)
- new net TH_CAM SDA: J2.4 (Pin_4), J3.3 (Pin_3)
